File: hardware/clock-divider.sch (KiCad schematic (older format))
At the start: 16 parts, among them J1 PWR, J2 Serial debug / programming he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, J3 SPI / ICSP header, U1 ATmega328P-PU, Y1 16MHz

Commit message: continue schematic
Parts:
- added D? (x2): 1N4148, Diode_THT:D_DO-35_SOD27_P7.62mm_Horizontal, symbol Diode:1N4148
- added Q? (x2): 2N3904, Package_TO_SOT_THT:TO-92_Inline, symbol Transistor_BJT:2N3904
- added R? (x2): 100k, symbol Device:R
- added U?: 74HC595, symbol 74xx:74HC595
Connections:
- net +5V: now also U?.10 (~SRCLR), U?.16 (VCC)
- net GND: now also D?.2 (A), D?.2 (A), Q?.1 (E), Q?.1 (E), U?.13 (~OE), U?.8 (GND)
- net DINA: now reaches U1.4 (PD2)
- net DINA: now also Q?.3 (C)
- net DINB: now reaches U1.5 (PD3)
- net DINB: now also Q?.3 (C)
- new net: D?.1 (K), Q?.2 (B), R?.1 (x2)
- new net CLKIN: R?.2
- new net RSTIN: R?.2
- new net S_CLK: U?.11 (SRCLK)
- new net S_DATA: U?.14 (SER)
- new net S_LATCH: U?.12 (RCLK)
- no-connect marks 0 -> 2
Other:
- note added: "Make use of internal pullups for inputs"
- moved on the sheet: C1, C2, C3, D1, R1, U1, Y1

Commit message: Added output protection
Parts:
- removed D4: 1N5817, Diode_THT:D_DO-41_SOD81_P10.16mm_Horizontal, symbol Diode:1N5817
- removed U?: 74HC595, symbol 74xx:74HC595
- added D10, D11, D12, D13, D6, D7, D8, D9: 1N4148, Diode_THT:D_DO-35_SOD27_P7.62mm_Horizontal, symbol Diode:1N4148
- added D14, D15, D16, D17, D18, D19, D20, D21: LED, symbol Device:LED
- added J10, J11, J4, J5, J6, J7, J8, J9: Conn_01x02, symbol Connector_Generic:Conn_01x02
- added J12: Conn_01x01, symbol Connector_Generic:Conn_01x01
- added Q10, Q3, Q4, Q5, Q6, Q7, Q8, Q9: 2N3904, Package_TO_SOT_THT:TO-92_Inline, symbol Transistor_BJT:2N3904
- added R10, R11, R12, R5, R6, R7, R8, R9: 33k, symbol Device:R
- added R13: 100k, symbol Device:R
- added R14, R15, R16, R17, R18, R19, R20, R21: 1k, symbol Device:R
- added R22, R23, R24, R25, R26, R27, R28, R29: 10k, symbol Device:R
- added R4: 47k, symbol Device:R
- added SW1: Divisions sets, symbol Switch:SW_SPDT_MSM
- added SW2: Trig / Gate, symbol Switch:SW_SPST
- gave numbers to parts that had none: 6
Connections:
- net GNDD is gone; now on net GND: J2.1 (Pin_1), J2.2 (Pin_2)
- net +12V: now also J1.9 (Pin_9), R4.1
- net +5V: now also J1.11 (Pin_11)
- net GND: now also D14.1 (K), D15.1 (K), D16.1 (K), D17.1 (K), D18.1 (K), D19.1 (K), D20.1 (K), D21.1 (K), J10.2 (Pin_2), J11.2 (Pin_2), J4.2 (Pin_2), J5.2 (Pin_2), J6.2 (Pin_2), J7.2 (Pin_2), J8.2 (Pin_2), J9.2 (Pin_2), R13.1, R22.1, R23.1, R24.1, R25.1, R26.1, R27.1, R28.1, R29.1, SW1.2, SW2.1 (A)
- net DIV6: now reaches U1.11 (PD5)
- net DIV6: now also R10.2
- net DIV7: now reaches U1.12 (PD6)
- net DIV7: now also R11.2
- net DIV8: now reaches U1.13 (PD7)
- net DIV8: now also R12.2
- net at U1.14 (PB0): now also SW1.3
- net at U1.15 (PB1): now also SW1.1
- net at U1.16 (PB2): now also SW2.2 (B)
- net ADCIN: now reaches U1.23 (PC0)
- net SPARE: now reaches U1.24 (PC1)
- net SPARE: now also J12.1 (Pin_1)
- net DIV1: now reaches U1.25 (PC2)
- net DIV1: now also R5.2
- net DIV2: now reaches U1.26 (PC3)
- net DIV2: now also R6.2
- net DIV3: now reaches U1.27 (PC4)
- net DIV3: now also R7.2
- net DIV4: now reaches U1.28 (PC5)
- net DIV4: now also R8.2
- net DIV5: now reaches U1.6 (PD4)
- net DIV5: now also R9.2
- net at J1.1 (Pin_1): no longer J1.2 (Pin_2)
- net at D3.2 (A), J1.10 (Pin_10): no longer J1.9 (Pin_9)
- net at D2.2 (A), J1.12 (Pin_12): no longer J1.11 (Pin_11)
- net at J1.13 (Pin_13): no longer J1.14 (Pin_14)
- net at J1.15 (Pin_15): no longer J1.16 (Pin_16)
- new net: D6.2 (A), Q3.1 (E), R14.1
- new net: Q3.2 (B), R5.1
- new net: Q10.3 (C), Q3.3 (C), Q4.3 (C), Q5.3 (C), Q6.3 (C), Q7.3 (C), Q8.3 (C), Q9.3 (C), R13.2, R4.2
- new net: D14.2 (A), R14.2
- new net: D6.1 (K), J4.1 (Pin_1), R22.2
- new net: D7.2 (A), Q4.1 (E), R15.1
- new net: Q4.2 (B), R6.1
- new net: D15.2 (A), R15.2
- new net: D7.1 (K), J5.1 (Pin_1), R23.2
- new net: D8.2 (A), Q5.1 (E), R16.1
- new net: Q5.2 (B), R7.1
- new net: D16.2 (A), R16.2
- new net: D8.1 (K), J6.1 (Pin_1), R24.2
- new net: D9.2 (A), Q6.1 (E), R17.1
- new net: Q6.2 (B), R8.1
- new net: D17.2 (A), R17.2
- new net: D9.1 (K), J7.1 (Pin_1), R25.2
- new net: D10.2 (A), Q7.1 (E), R18.1
- new net: Q7.2 (B), R9.1
- new net: D18.2 (A), R18.2
- new net: D10.1 (K), J8.1 (Pin_1), R26.2
- new net: D11.2 (A), Q8.1 (E), R19.1
- new net: Q8.2 (B), R10.1
- new net: D19.2 (A), R19.2
- new net: D11.1 (K), J9.1 (Pin_1), R27.2
- new net: D12.2 (A), Q9.1 (E), R20.1
- new net: Q9.2 (B), R11.1
- new net: D20.2 (A), R20.2
- new net: D12.1 (K), J10.1 (Pin_1), R28.2
- new net: D13.2 (A), Q10.1 (E), R21.1
- new net: Q10.2 (B), R12.1
- new net: D21.2 (A), R21.2
- new net: D13.1 (K), J11.1 (Pin_1), R29.2
- no-connect marks 2 -> 7
Other:
- moved on the sheet: C1, C2, C3, D1, R1, U1, Y1

Commit message: Labelling
Other:
- note added: "Make use of internal pullups for digital inputs"
- note added: "Power"
- note added: "Programming / debuging headers"
- note removed: "Make use of internal pullups for inputs"
Changed lines of the file:
@@
 Wire Wire Line
 	2050 3750 2200 3750
-Text Notes 1100 5300 0    50   ~ 0
-Make use of internal pullups for inputs
+Text Notes 1050 5250 0    50   ~ 0
+Make use of internal pullups for digital inputs
 NoConn ~ 850  1850
 Text GLabel 2200 2750 2    50   Input ~ 0
@@
 	1    0    0    -1
 $EndComp
+Text Notes 7800 800  0    100  ~ 0
+Programming / debuging headers
+Text Notes 7550 2500 0    100  ~ 0
+Power
 $EndSCHEMATC
